File: PCB/LatticePCB.kicad_pcb (KiCad board)
At the start: 2 copper layers, 64.1 x 35.1 mm, 23 parts, among them M1 M1, M2 M2, M3 M3, U1 Teensy++1.0_(Arduino), U2 AMS1117CS-5.0

Commit message: Yeet
Other:
- board text added: "ACCELEROMETER LIS311DLH"
- board text added: "L.UEDA"
- board text added: "LATTICE BOARD V1"
- board text added: "TEENSY 4.0"

Commit message: Balance chargine ports added
Parts:
- added J1: Conn_01x03_Pin, Connector_JST:JST_XH_B3B-XH-A_1x03_P2.50mm_Vertical, F.Cu at (143.1, 94.1)
- added J2: Conn_01x03_Pin, Connector_JST:JST_XH_B3B-XH-A_1x03_P2.50mm_Vertical, F.Cu at (130.2, 94.0)
- added J3: Conn_01x05_Pin, Connector_JST:JST_XH_B5B-XH-A_1x05_P2.50mm_Vertical, F.Cu at (108.6, 94.0)
Routing:
- net Net-(J1-Pin_2): track 0.00 -> 33.1 mm
- net Net-(J1-Pin_1): track 0.00 -> 31.7 mm
- net Net-(J1-Pin_3): track 0.00 -> 31.0 mm
- net Net-(J2-Pin_2): track 0.00 -> 23.7 mm
- net Net-(J2-Pin_1): track 0.00 -> 23.0 mm
Other:
- board text added: "- - -"
- board text added: "1"
- board text added: "2"
- board text added: "["
- board text added: "]"
- board text removed: "LATTICE"
