File: PCB/LatticePCB.kicad_sch (KiCad schematic)
At the start: 3 parts, among them U1 Teensy++1.0_(Arduino), U2 AMS1117CS-5.0

Commit message: Balance chargine ports added
Parts:
- added J1, J2: Conn_01x03_Pin, Connector_JST:JST_XH_B3B-XH-A_1x03_P2.50mm_Vertical, symbol Connector:Conn_01x03_Pin
- added J3: Conn_01x05_Pin, Connector_JST:JST_XH_B5B-XH-A_1x05_P2.50mm_Vertical, symbol Connector:Conn_01x05_Pin
Connections:
- new net: J2.1 (Pin_1), J3.1 (Pin_1)
- new net: J2.2 (Pin_2), J3.2 (Pin_2)
- new net: J1.1 (Pin_1), J3.3 (Pin_3)
- new net: J1.2 (Pin_2), J3.4 (Pin_4)
- new net: J1.3 (Pin_3), J3.5 (Pin_5)
Changed lines of the file:
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@@
 (kicad_sch (version 20230121) (generator eeschema)
   (paper "A4")
+  (wire (pts (xy 236.22 100.33) (xy 250.19 100.33))
+    (stroke (width 0) (type default))
+  )
   (wire (pts (xy 78.74 78.74) (xy 78.74 110.49))
     (stroke (width 0) (type default))
   )
+  (wire (pts (xy 250.19 87.63) (xy 255.27 87.63))
+    (stroke (width 0) (type default))
+  )
   (wire (pts (xy 76.2 73.66) (xy 87.63 73.66))
     (stroke (width 0) (type default))
@@
     (stroke (width 0) (type default))
   )
+  (wire (pts (xy 236.22 85.09) (xy 262.89 85.09))
+    (stroke (width 0) (type default))
+  )
+  (wire (pts (xy 252.73 90.17) (xy 252.73 92.71))
+    (stroke (width 0) (type default))
+  )
+  (wire (pts (xy 236.22 80.01) (xy 257.81 80.01))
+    (stroke (width 0) (type default))
+  )
   (wire (pts (xy 135.89 105.41) (xy 135.89 123.19))
     (stroke (width 0) (type default))
@@
     (stroke (width 0) (type default))
   )
+  (wire (pts (xy 236.22 97.79) (xy 247.65 97.79))
+    (stroke (width 0) (type default))
+  )
+  (wire (pts (xy 250.19 100.33) (xy 250.19 87.63))
+    (stroke (width 0) (type default))
+  )
   (wire (pts (xy 97.79 107.95) (xy 85.09 107.95))
     (stroke (width 0) (type default))
@@
     (stroke (width 0) (type default))
   )
+  (wire (pts (xy 247.65 90.17) (xy 252.73 90.17))
+    (stroke (width 0) (type default))
+  )
   (wire (pts (xy 85.09 107.95) (xy 85.09 76.2))
     (stroke (width 0) (type default))
@@
     (stroke (width 0) (type default))
   )
+  (wire (pts (xy 257.81 80.01) (xy 257.81 92.71))
+    (stroke (width 0) (type default))
+  )
+  (wire (pts (xy 247.65 97.79) (xy 247.65 90.17))
+    (stroke (width 0) (type default))
+  )
   (wire (pts (xy 133.35 105.41) (xy 135.89 105.41))
     (stroke (width 0) (type default))
   )
+  (wire (pts (xy 260.35 92.71) (xy 260.35 82.55))
+    (stroke (width 0) (type default))
+  )
+  (wire (pts (xy 236.22 82.55) (xy 260.35 82.55))
+    (stroke (width 0) (type default))
+  )
+  (wire (pts (xy 255.27 87.63) (xy 255.27 92.71))
+    (stroke (width 0) (type default))
+  )
+  (wire (pts (xy 262.89 85.09) (xy 262.89 92.71))
+    (stroke (width 0) (type default))
+  )
   (symbol (lib_id "power:GNDREF") (at 80.01 55.88 0) (unit 1)
     (in_bom yes) (on_board yes) (dnp no) (fields_autoplaced)
@@
     (pin "1")
     (instances
-      (project "Tessellate2"
+      (project "LatticePCB"
         (path "/bd2eed61-2285-4a26-8727-12a0d3a662a6"
           (reference "#PWR0101") (unit 1)
@@
     )
   )
+  (symbol (lib_id "Connector:Conn_01x05_Pin") (at 257.81 97.79 90) (unit 1)
+    (in_bom yes) (on_board yes) (dnp no) (fields_autoplaced)
+    (property "Reference" "J3" (at 257.81 100.33 90)
+      (effects (font (size 1.27 1.27)))
+    )
+    (property "Value" "Conn_01x05_Pin" (at 257.81 102.87 90)
+      (effects (font (size 1.27 1.27)))
+    )
+    (property "Footprint" "Connector_JST:JST_XH_B5B-XH-A_1x05_P2.50mm_Vertical" (at 257.81 97.79 0)
+      (effects (font (size 1.27 1.27)) hide)
+    )
+    (property "Datasheet" "~" (at 257.81 97.79 0)
+      (effects (font (size 1.27 1.27)) hide)
+    )
+    (pin "1")
+    (pin "2")
+    (pin "3")
+    (pin "4")
+    (pin "5")
+    (instances
+      (project "LatticePCB"
+        (path "/bd2eed61-2285-4a26-8727-12a0d3a662a6"
+          (reference "J3") (unit 1)
+        )
+      )
+    )
+  )
+  (symbol (lib_id "Connector:Conn_01x03_Pin") (at 231.14 100.33 0) (unit 1)
+    (in_bom yes) (on_board yes) (dnp no) (fields_autoplaced)
+    (property "Reference" "J2" (at 231.775 93.98 0)
+      (effects (font (size 1.27 1.27)))
+    )
+    (property "Value" "Conn_01x03_Pin" (at 231.775 96.52 0)
+      (effects (font (size 1.27 1.27)) hide)
+    )
+    (property "Footprint" "Connector_JST:JST_XH_B3B-XH-A_1x03_P2.50mm_Vertical" (at 231.14 100.33 0)
+      (effects (font (size 1.27 1.27)) hide)
+    )
+    (property "Datasheet" "~" (at 231.14 100.33 0)
+      (effects (font (size 1.27 1.27)) hide)
+    )
+    (pin "1")
+    (pin "2")
+    (pin "3")
+    (instances
+      (project "LatticePCB"
+        (path "/bd2eed61-2285-4a26-8727-12a0d3a662a6"
+          (reference "J2") (unit 1)
+        )
+      )
+    )
+  )
   (symbol (lib_id "power:GNDREF") (at 88.9 48.26 0) (unit 1)
     (in_bom yes) (on_board yes) (dnp no) (fields_autoplaced)
@@
     (pin "1")
     (instances
-      (project "Tessellate2"
+      (project "LatticePCB"
         (path "/bd2eed61-2285-4a26-8727-12a0d3a662a6"
           (reference "#PWR02") (unit 1)
@@
     (pin "8")
     (instances
-      (project "Tessellate2"
+      (project "LatticePCB"
         (path "/bd2eed61-2285-4a26-8727-12a0d3a662a6"
           (reference "LIS331DLH1") (unit 1)
@@
     (pin "1")
     (instances
-      (project "Tessellate2"
+      (project "LatticePCB"
         (path "/bd2eed61-2285-4a26-8727-12a0d3a662a6"
           (reference "#PWR01") (unit 1)
@@
     (pin "1")
     (instances
-      (project "Tessellate2"
+      (project "LatticePCB"
         (path "/bd2eed61-2285-4a26-8727-12a0d3a662a6"
           (reference "#PWR04") (unit 1)
@@
     (pin "8")
     (instances
-      (project "Tessellate2"
+      (project "LatticePCB"
         (path "/bd2eed61-2285-4a26-8727-12a0d3a662a6"
           (reference "U2") (unit 1)
@@
     (pin "9")
     (instances
-      (project "Tessellate2"
+      (project "LatticePCB"
         (path "/bd2eed61-2285-4a26-8727-12a0d3a662a6"
           (reference "U1") (unit 1)
@@
     (pin "1")
     (instances
-      (project "Tessellate2"
+      (project "LatticePCB"
         (path "/bd2eed61-2285-4a26-8727-12a0d3a662a6"
           (reference "#PWR03") (unit 1)
         )
       )
+    )
+  )
+  (symbol (lib_id "Connector:Conn_01x03_Pin") (at 231.14 82.55 0) (unit 1)
+    (in_bom yes) (on_board yes) (dnp no) (fields_autoplaced)
+    (property "Reference" "J1" (at 231.775 76.2 0)
+      (effects (font (size 1.27 1.27)))
+    )
+    (property "Value" "Conn_01x03_Pin" (at 231.775 78.74 0)
+      (effects (font (size 1.27 1.27)))
+    )
+    (property "Footprint" "Connector_JST:JST_XH_B3B-XH-A_1x03_P2.50mm_Vertical" (at 231.14 82.55 0)
+      (effects (font (size 1.27 1.27)) hide)
+    )
+    (property "Datasheet" "~" (at 231.14 82.55 0)
+      (effects (font (size 1.27 1.27)) hide)
+    )
+    (pin "1")
+    (pin "2")
+    (pin "3")
+    (instances
+      (project "LatticePCB"
+        (path "/bd2eed61-2285-4a26-8727-12a0d3a662a6"
+          (reference "J1") (unit 1)
+        )
+      )
